File: DragonUSBHost.brd (EAGLE design)
At the start: 49.5 x 59.7 mm, 30 parts, among them IC1 MAX3421EEHJ, J1 Dragino, J2 MICROSD, J3 Sensors, J4 Serial, J5 XBee, P1 USB_, Q1 12 MHz

Commit message: foo
Parts:
- moved LED1 46.9 mm to (48.9, 49.2), turned to 0 degrees
- moved LED3 46.5 mm to (48.9, 52.4), turned to 0 degrees
- moved LED2 46.4 mm to (48.9, 45.7), turned to 0 degrees
- moved R4 39.8 mm to (45.4, 49.2), turned to 180 degrees
- moved R11 38.9 mm to (45.4, 52.4), turned to 180 degrees
- moved R5 38.7 mm to (45.4, 45.7), turned to 180 degrees
- moved P1 32.4 mm to (9.53, 48.9), turned to 0 degrees
- moved L2 32.1 mm to (7.62, 40.3)
- moved J5 26.0 mm to (38.7, 27.6)
- moved F1 24.9 mm to (24.4, 56.2), turned to 0 degrees
- moved R2 24.1 mm to (44.5, 12.7)
- moved J1 24.1 mm to (36.8, 6.35)
- moved J3 24.1 mm to (36.8, 56.3)
- moved J4 24.1 mm to (36.8, 2.54)
- moved R3 24.1 mm to (41.9, 12.7)
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Routing:
- net +5V: track 51.0 -> 79.9 mm, vias 3 -> 2
- net !USB_CS: track 44.4 -> 70.5 mm, vias 2 -> 5
- net +3V3: track 151.7 -> 133.1 mm, vias 7 -> 1
- net !INTERRUPT: track 4.76 -> 23.2 mm
- net N$13: track 18.0 -> 31.6 mm
- net SCK: track 85.7 -> 72.9 mm, vias 4 -> 3
- net N$9: track 33.4 -> 21.3 mm, vias 2 -> 0
- net TXD: track 49.8 -> 40.8 mm
- net RXD: track 51.3 -> 42.8 mm
- net MISO: track 78.9 -> 71.5 mm, vias 4 -> 3
- net !RESET: track 5.68 -> 10.6 mm
- net !SDCARD_CS: track 54.5 -> 50.2 mm
- net N$4: track 8.62 -> 5.13 mm
- net N$2: track 7.68 -> 4.72 mm
- net N$12: track 4.15 -> 1.69 mm
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Other:
- outline, holes or cut-outs redrawn
- board text added: "10k"
- board text added: "USB Host Port"
- board text removed: "USBHost Port"

Commit message: foo
Routing:
- net MOSI: track 68.7 -> 73.5 mm
Other:
- board text removed: "10k"
Changed lines of the file:
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@@
 <wire x1="51.435" y1="2.54" x2="51.435" y2="57.15" width="0" layer="20"/>
 <wire x1="51.435" y1="57.15" x2="48.895" y2="59.69" width="0" layer="20" curve="90"/>
-<text x="22.225" y="44.45" size="0.8128" layer="21" ratio="15">10k</text>
 </plain>
 <attributes>
@@
 </element>
 <element name="R8" library="freetronics-master-v1" package="0805" value="10k" x="20.6375" y="45.085" smashed="yes">
-<attribute name="VALUE" x="31.75" y="22.5425" size="0.8128" layer="27" ratio="15"/>
+<attribute name="VALUE" x="22.225" y="44.45" size="0.8128" layer="27" ratio="15"/>
 </element>
 <element name="Q1" library="freetronics-master-v1" package="HC49US" value="12 MHz" x="22.86" y="41.275" smashed="yes">
@@
 <wire x1="11.29" y1="35.7" x2="12.7" y2="34.29" width="0.4064" layer="1"/>
 <via x="12.7" y="34.29" extent="1-16" drill="0.4"/>
-<wire x1="12.7" y1="34.29" x2="12.7" y2="35.56" width="0.2032" layer="16"/>
-<wire x1="12.7" y1="35.56" x2="26.035" y2="48.895" width="0.2032" layer="16"/>
-<wire x1="26.035" y1="48.895" x2="27.305" y2="48.895" width="0.2032" layer="16"/>
-<wire x1="27.305" y1="48.895" x2="27.94" y2="49.53" width="0.2032" layer="16"/>
-<wire x1="12.7" y1="34.29" x2="12.7" y2="32.385" width="0.2032" layer="16"/>
-<wire x1="12.7" y1="32.385" x2="13.335" y2="31.75" width="0.2032" layer="16"/>
-<wire x1="13.335" y1="31.75" x2="17.145" y2="31.75" width="0.2032" layer="16"/>
-<wire x1="17.145" y1="31.75" x2="25.4" y2="23.495" width="0.2032" layer="16"/>
+<wire x1="12.7" y1="34.29" x2="12.7" y2="35.56" width="0.4064" layer="16"/>
+<wire x1="12.7" y1="35.56" x2="25.4" y2="48.26" width="0.4064" layer="16"/>
+<wire x1="25.4" y1="48.26" x2="26.67" y2="48.26" width="0.4064" layer="16"/>
+<wire x1="26.67" y1="48.26" x2="27.94" y2="49.53" width="0.4064" layer="16"/>
+<wire x1="12.7" y1="34.29" x2="12.7" y2="32.385" width="0.4064" layer="16"/>
+<wire x1="12.7" y1="32.385" x2="13.335" y2="31.75" width="0.4064" layer="16"/>
+<wire x1="13.335" y1="31.75" x2="17.145" y2="31.75" width="0.4064" layer="16"/>
+<wire x1="17.145" y1="31.75" x2="25.4" y2="23.495" width="0.4064" layer="16"/>
 <wire x1="25.4" y1="23.495" x2="25.4" y2="17.78" width="0.2032" layer="16"/>
 <wire x1="25.4" y1="17.78" x2="27.305" y2="15.875" width="0.2032" layer="16"/>
@@
 <wire x1="26.19" y1="50.645" x2="26.67" y2="50.165" width="0.2032" layer="1"/>
 <via x="26.67" y="50.165" extent="1-16" drill="0.4"/>
-<wire x1="26.67" y1="50.165" x2="11.43" y2="34.925" width="0.2032" layer="16"/>
 <wire x1="11.43" y1="34.925" x2="11.43" y2="30.48" width="0.2032" layer="16"/>
 <via x="11.43" y="30.48" extent="1-16" drill="0.4"/>
@@
 <wire x1="11.43" y1="30.48" x2="17.145" y2="30.48" width="0.4064" layer="16"/>
 <wire x1="17.145" y1="30.48" x2="24.765" y2="22.86" width="0.4064" layer="16"/>
+<wire x1="26.67" y1="50.165" x2="26.035" y2="49.53" width="0.4064" layer="16"/>
+<wire x1="26.035" y1="49.53" x2="25.4" y2="49.53" width="0.4064" layer="16"/>
+<wire x1="25.4" y1="49.53" x2="11.43" y2="35.56" width="0.4064" layer="16"/>
+<wire x1="11.43" y1="35.56" x2="11.43" y2="30.48" width="0.4064" layer="16"/>
 </signal>
 <signal name="SCK">
@@
 <wire x1="21.59" y1="27.305" x2="12.7" y2="27.305" width="0.4064" layer="1"/>
 <wire x1="12.7" y1="27.305" x2="10.16" y2="29.845" width="0.4064" layer="16"/>
-<wire x1="10.16" y1="29.845" x2="10.16" y2="34.925" width="0.4064" layer="16"/>
-<wire x1="10.16" y1="34.925" x2="22.86" y2="47.625" width="0.4064" layer="16"/>
-<wire x1="22.86" y1="47.625" x2="22.86" y2="54.61" width="0.4064" layer="16"/>
+<wire x1="10.16" y1="29.845" x2="10.16" y2="36.195" width="0.4064" layer="16"/>
+<wire x1="10.16" y1="36.195" x2="22.86" y2="48.895" width="0.4064" layer="16"/>
+<wire x1="22.86" y1="48.895" x2="22.86" y2="54.61" width="0.4064" layer="16"/>
 <wire x1="22.86" y1="54.61" x2="24.4475" y2="56.1975" width="0.4064" layer="16"/>
 <via x="24.4475" y="56.1975" extent="1-16" drill="0.4"/>
