File: DragonUSBHost.brd (EAGLE design)
At the start: 49.5 x 59.7 mm, 30 parts, among them IC1 MAX3421EEHJ, J1 Dragino, J2 MICROSD, J3 Sensors, J4 Serial, J5 XBee, P1 USB_, Q1 12 MHz

Commit message: foo
Parts:
- added U$21: (no value), OSHW:OSHW_6X100_NOTEXT
Changed lines of the file:
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@@
 <text x="19.52625" y="46.0375" size="0.8128" layer="21" ratio="15">33R</text>
 <text x="3.96875" y="36.03625" size="0.8128" layer="21" ratio="15" rot="SR270">MICRO SD CARD</text>
-<text x="29.845" y="26.035" size="1.016" layer="21" ratio="15">smartenergygroups.com</text>
-<text x="29.21" y="24.765" size="0.8636" layer="21" ratio="15">Dragon USB Host Controller</text>
-<text x="29.5275" y="18.7325" size="0.7874" layer="21" ratio="15">Luke Weston, 2012</text>
+<text x="29.845" y="31.115" size="1.016" layer="21" ratio="15">smartenergygroups.com</text>
+<text x="29.21" y="29.845" size="0.8636" layer="21" ratio="15">Dragon USB Host Controller</text>
+<text x="29.5275" y="23.8125" size="0.7874" layer="21" ratio="15">Luke Weston, 2012</text>
 <text x="29.5275" y="17.4625" size="0.762" layer="21" ratio="15">Released under the CERN Open</text>
 <text x="28.2575" y="16.1925" size="0.762" layer="21" ratio="15">Hardware License: ohwr.org/cernohl</text>
-<text x="29.5275" y="22.5425" size="0.8128" layer="21" ratio="15">AR2317 GPIO {0, 1, 2, 3, 4}</text>
-<text x="29.21" y="20.955" size="0.8128" layer="21" ratio="15">= {MISO, MOSI, SCK, !Sd!, !USB!}</text>
+<text x="29.5275" y="27.6225" size="0.8128" layer="21" ratio="15">AR2317 GPIO {0, 1, 2, 3, 4}</text>
+<text x="29.21" y="26.035" size="0.8128" layer="21" ratio="15">= {MISO, MOSI, SCK, !Sd!, !USB!}</text>
 <text x="29.5275" y="0.3175" size="0.8128" layer="21" ratio="15">GND</text>
 <text x="32.0675" y="0.3175" size="0.8128" layer="21" ratio="15">12V</text>
@@
 <attribute name="VALUE" x="44.7675" y="44.1325" size="0.8128" layer="27" ratio="15"/>
 </element>
+<element name="U$21" library="OSHW" package="OSHW_6X100_NOTEXT" value="" x="37.465" y="18.415"/>
 </elements>
 <signals>
