File: DragonUSBHost.sch (EAGLE design)
At the start: 30 parts, among them IC1 MAX3421EEHJ, J1 Dragino, J2 MICROSD, J3 Sensors, J4 Serial, J5 XBee, P1 USB_, Q1 12 MHz

Commit message: foo
Parts:
- Q1: value 12 MHz -> 12MHz; device freetronics-master-v1:CRYSTALHC49US -> SparkFun:CRYSTAL5X3
- R11, R4, R5: value 1k -> 330R
Other:
- note added: "5x3.2mm"
- note added: "CTX819CT-ND"
- note removed: "HC49US"
Changed lines of the file:
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@@
 <setting verticaltext="up"/>
 </settings>
-<grid distance="0.1" unitdist="inch" unit="inch" style="lines" multiple="1" display="no" altdistance="0.01" altunitdist="inch" altunit="inch"/>
+<grid distance="0.1" unitdist="inch" unit="inch" style="lines" multiple="1" display="yes" altdistance="0.01" altunitdist="inch" altunit="inch"/>
 <layers>
 <layer number="1" name="Top" color="4" fill="1" visible="no" active="no"/>
@@
 <part name="U$16" library="freetronics-luke" deviceset="+3.3V" device=""/>
 <part name="C3" library="freetronics-master-v1" deviceset="CAP" device="0805" value="22pF"/>
-<part name="R11" library="freetronics-master-v1" deviceset="RESISTOR" device="0805" value="1k"/>
+<part name="R11" library="freetronics-master-v1" deviceset="RESISTOR" device="0805" value="330R"/>
 <part name="LED3" library="freetronics-master-v1" deviceset="LED" device="0805" value="Power"/>
 <part name="C4" library="freetronics-master-v1" deviceset="CAP" device="0805" value="22pF"/>
@@
 <part name="R7" library="freetronics-master-v1" deviceset="RESISTOR" device="0805" value="10k"/>
 <part name="R8" library="freetronics-master-v1" deviceset="RESISTOR" device="0805" value="10k"/>
-<part name="Q1" library="freetronics-master-v1" deviceset="CRYSTAL" device="HC49US" value="12 MHz"/>
 <part name="F1" library="freetronics-luke" deviceset="PTC" device="" value="500mA"/>
 <part name="C2" library="freetronics-master-v1" deviceset="CAP" device="0805" value="100nF"/>
@@
 <part name="LED1" library="freetronics-master-v1" deviceset="LED" device="0805" value="RSSI"/>
 <part name="LED2" library="freetronics-master-v1" deviceset="LED" device="0805" value="Assoc"/>
-<part name="R4" library="freetronics-master-v1" deviceset="RESISTOR" device="0805" value="1k"/>
-<part name="R5" library="freetronics-master-v1" deviceset="RESISTOR" device="0805" value="1k"/>
+<part name="R4" library="freetronics-master-v1" deviceset="RESISTOR" device="0805" value="330R"/>
+<part name="R5" library="freetronics-master-v1" deviceset="RESISTOR" device="0805" value="330R"/>
 <part name="U$9" library="freetronics-luke" deviceset="GND" device=""/>
 <part name="P+3" library="supply1" deviceset="+12V" device=""/>
@@
 <part name="U$20" library="freetronics-luke" deviceset="GND" device=""/>
 <part name="P+4" library="supply1" deviceset="+12V" device=""/>
+<part name="Q1" library="SparkFun" deviceset="CRYSTAL" device="5X3" value="12MHz"/>
 </parts>
 <sheets>
@@
 <text x="121.92" y="116.84" size="1.27" layer="98">0805</text>
 <text x="170.18" y="116.84" size="1.27" layer="98">32-TQFP</text>
-<text x="134.62" y="76.2" size="1.27" layer="98">HC49US</text>
+<text x="133.35" y="76.2" size="1.27" layer="98">5x3.2mm</text>
 <text x="58.42" y="78.74" size="1.27" layer="98">0805</text>
 <text x="63.5" y="124.46" size="1.27" layer="98">0805</text>
@@
 <text x="193.04" y="337.82" size="1.27" layer="98">Amphenol 101-00660-68-6</text>
 <text x="193.04" y="335.28" size="1.27" layer="98">Digi-Key 101-00660-68-6-1-ND</text>
+<text x="118.11" y="73.66" size="1.27" layer="98">CTX819CT-ND</text>
 </plain>
 <instances>
@@
 <attribute name="NAME" x="142.24" y="121.92" size="1.27" layer="95"/>
 <attribute name="VALUE" x="142.24" y="119.38" size="1.27" layer="96"/>
-</instance>
-<instance part="Q1" gate="G$1" x="137.16" y="73.66" smashed="yes" rot="R180">
-<attribute name="NAME" x="127" y="73.66" size="1.27" layer="95"/>
-<attribute name="VALUE" x="134.62" y="78.74" size="1.27" layer="96"/>
 </instance>
 <instance part="F1" gate="G$1" x="96.52" y="134.62" smashed="yes">
@@
 <attribute name="VALUE" x="99.06" y="340.36" size="1.27" layer="96"/>
 </instance>
+<instance part="Q1" gate="G$1" x="137.16" y="73.66" smashed="yes" rot="R180">
+<attribute name="NAME" x="137.16" y="68.58" size="1.27" layer="95"/>
+<attribute name="VALUE" x="133.35" y="78.74" size="1.27" layer="96"/>
+</instance>
 </instances>
